File: Hardware/QuadMod.kicad_sch (KiCad schematic)
At the start: 98 parts, among them J2 Eurorack_10_pin_power, J6 SWD_Header, U1 STM32H563VIT, U2 MCP6004, U3 MCP6004, U4 AK4619VN, U5 TL074, U6 LM1117-3.3, U7 LM1117-5.0, Y1 8MHz 20pF

Commit message: Phaser filter count can be set to any number between 1 and 16
Parts:
- added Q1: MMBT3904, Package_TO_SOT_SMD:SOT-23, symbol Transistor_BJT:MMBT3904
- added R32, R33: 4k7, Resistor_SMD:R_0603_1608Metric, symbol Device:R_Small
- added unit 3 of U3
Connections:
- net +3V3: now also R33.2
- net GND: now also Q1.2 (E)
- new net: Q1.1 (B), R32.2
- new net CLOCK: U3.10 (+)
- new net CLOCK_SCALED: U3.8, U3.9 (-)
- new net MIDI_IN: R32.1
- new net MIDI_UART: Q1.3 (C), R33.1
Other:
- note added: "UART4_RX"
- moved on the sheet: R1, R5, R6, R7, U3B

Commit message: Started roughing out panel design
Parts:
- added J3, J4, J5, J6: Conn_01x12_Pin, symbol Connector:Conn_01x12_Pin
- added R1 (x8): 75k, Resistors_SMD:R_0603_HandSoldering, symbol Device:R
- added R5 (x8): 91k, Resistors_SMD:R_0603_HandSoldering, symbol Device:R
- added R6 (x8), R7 (x8): 47k, Resistors_SMD:R_0603_HandSoldering, symbol Device:R
- added U3 (x8): MCP6004, SMD_Packages:SOIC-14_N, symbol Amplifier_Operational:MCP6004
Connections:
- net WET_DRY_MIX is gone; now on net DLY_MIX: R6.1, U3.7
- net -5V_REF: now also R1.2, R1.2, R1.2, R1.2, R1.2, R1.2, R1.2, R1.2
- net GND: now also U3.5 (+), U3.5 (+), U3.5 (+), U3.5 (+), U3.5 (+), U3.5 (+), U3.5 (+), U3.5 (+)
- net LFO_RANGE: now reaches U1.15 (PC0)
- net LFO_RANGE: now also R6.1, U3.7
- net DLY_TIME: now reaches U1.16 (PC1)
- net DLY_TIME: now also R6.1, U3.7
- net FX_MIX: now reaches U1.17 (PC2_C)
- net FX_MIX: now also R6.1, U3.7
- net FX_FEEDBACK: now reaches U1.18 (PC3_C)
- net FX_FEEDBACK: now also R6.1, U3.7
- net DLY_FILTER: now reaches U1.32 (PA7)
- net DLY_FILTER: now also R6.1, U3.7
- net LFO_SPEED: now reaches U1.33 (PC4)
- net LFO_SPEED: now also R6.1, U3.7
- net DLY_MIX: now reaches U1.34 (PC5)
- net DLY_FEEDBACK: now reaches U1.35 (PB0)
- net DLY_FEEDBACK: now also R6.1, U3.7
- net LFO_BASEFREQ: now reaches U1.36 (PB1)
- net LFO_BASEFREQ: now also R6.1, U3.7
- net MIX_CV renamed DLY_MIX_CV
- net DLY_MIX_CV: now also J3.1 (Pin_1)
- net MIX_POT renamed DLY_MIX_POT
- net DLY_MIX_POT: now also J3.2 (Pin_2)
- new net: R1.1, R5.1, R6.2, R7.1, U3.6 (-) (x8)
- new net CLOCK_IN: J4.8 (Pin_8)
- new net DLY_FEEDBACK_CV: J3.5 (Pin_5), R5.2
- new net DLY_FEEDBACK_POT: J3.6 (Pin_6), R7.2
- new net DLY_FILTER_CV: J3.9 (Pin_9), R5.2
- new net DLY_FILTER_POT: J3.10 (Pin_10), R7.2
- new net DLY_TIME_CV: J3.7 (Pin_7), R5.2
- new net DLY_TIME_POT: J3.8 (Pin_8), R7.2
- new net FX_FEEDBACK_CV: J4.3 (Pin_3), R5.2
- new net FX_FEEDBACK_POT: J4.4 (Pin_4), R7.2
- new net FX_MIX_CV: J3.3 (Pin_3), R5.2
- new net FX_MIX_POT: J3.4 (Pin_4), R7.2
- new net FX_TYPE: J4.7 (Pin_7)
- new net LFO_BASEFREQ_CV: J4.5 (Pin_5), R5.2
- new net LFO_BASEFREQ_POT: J4.6 (Pin_6), R7.2
- new net LFO_RANGE_CV: J4.1 (Pin_1), R5.2
- new net LFO_RANGE_POT: J4.2 (Pin_2), R7.2
- new net LFO_SPEED_CV: J3.11 (Pin_11), R5.2
- new net LFO_SPEED_POT: J3.12 (Pin_12), R7.2
Other:
- moved on the sheet: R1, R5, R6, R7, U3B
