File: Hardware/QuadMod Components.kicad_sch (KiCad schematic)
At the start: 145 parts, among them J2 Eurorack_10_pin_power, J3 Conn_01x12_Pin, J4 Conn_01x12_Pin, J5 Conn_01x12_Pin, J6 Conn_01x12_Pin, J6 SWD_Header, Q1 MMBT3904, U1 STM32H563VIT, U2 MCP6004, U3 MCP6004, U4 AK4619VN, U5 TL074, U6 LM1117-3.3, U7 LM1117-5.0, Y1 8MHz 20pF

Commit message: Cleaned up schematic
Parts:
- removed C17, C18: 1uF, Capacitor_SMD:C_0603_1608Metric_Pad1.08x0.95mm_HandSolder, symbol Device:C_Small
- removed C23: 10uF, Capacitor_SMD:C_1206_3216Metric, symbol Encoder:CP_Small
- removed C24: 22uF, Capacitor_SMD:CP_Elec_4x5.8, symbol Encoder:CP_Small
- removed C43: 10uF, Capacitor_SMD:C_1206_3216Metric, symbol Device:C
- removed C45: 22uF, Capacitor_SMD:CP_Elec_4x5.8, symbol Device:C
- removed J3, J4, J5, J6: Conn_01x12_Pin, symbol Connector:Conn_01x12_Pin
- removed J6: SWD_Header, Custom_Footprints:SWD_header, symbol Connector:Conn_01x04_Male
- removed Q1: MMBT3904, Package_TO_SOT_SMD:SOT-23, symbol Transistor_BJT:MMBT3904
- removed R1 (x4): 75k, Resistors_SMD:R_0603_HandSoldering, symbol Device:R
- removed R21, R22: 390k, Resistor_SMD:R_0603_1608Metric_Pad0.98x0.95mm_HandSolder, symbol Device:R
- removed R23, R24: 10k, Resistor_SMD:R_0603_1608Metric_Pad0.98x0.95mm_HandSolder, symbol Device:R
- removed R27, R28: 14k, Resistor_SMD:R_0603_1608Metric_Pad0.98x0.95mm_HandSolder, symbol Device:R
- removed R5 (x4): 91k, Resistors_SMD:R_0603_HandSoldering, symbol Device:R
- removed R6 (x4), R7 (x4): 47k, Resistors_SMD:R_0603_HandSoldering, symbol Device:R
- removed U3 (x5): MCP6004, SMD_Packages:SOIC-14_N, symbol Amplifier_Operational:MCP6004
- removed unit 3 of U3
- removed U5: TL074, Package_SO:SO-14_3.9x8.65mm_P1.27mm, symbol Amplifier_Operational:TL074
- removed U6: LM1117-3.3, Package_TO_SOT_SMD:SOT-223-3_TabPin2, symbol Regulator_Linear:LM1117-3.3
- removed U7: LM1117-5.0, Package_TO_SOT_SMD:SOT-223-3_TabPin2, symbol Regulator_Linear:LM1117-5.0
- added C38: 100nF, Capacitor_SMD:C_0805_2012Metric, symbol Device:C_Small
- added C39, C40: 10uF, Capacitor_SMD:C_0805_2012Metric, symbol Device:C_Small
- added C41: 22uF, Capacitor_SMD:CP_Elec_4x5.8, symbol Device:C_Polarized_Small
- added C42: 47uF, Resistor_SMD:R_1206_3216Metric, symbol Device:C_Small
- added J1, J2, J3, J4: Conn_01x08_Pin, symbol Connector:Conn_01x08_Pin
- added J7: Prog_Header, symbol Connector:Conn_01x04_Pin
- added J7: USB_B_Micro, Custom_Footprints:USB_Micro-B_Amphenol, symbol Connector:USB_B_Micro
- added J8: Extra_Outs, symbol Connector:Conn_01x02_Pin
- added L2: L, Inductor_SMD:L_0805_2012Metric, symbol Device:L
- added R17, R19: 1k, Resistor_SMD:R_0603_1608Metric, symbol Device:R_Small
- added U1: STF202-22T1G, Custom_Footprints:STF202-22T1G, symbol STF202-22T1G:STF202-22T1G
- added U6: TL072, symbol Amplifier_Operational:TL072
- added U7: MCP6002-xSN, symbol Amplifier_Operational:MCP6002-xSN
- added U7: LD1117-3.3-4Tab, TO_SOT_Packages_SMD:SOT-223-3_TabPin2, symbol LD1117-3.3-4Tab:LD1117-3.3-4Tab
- L1: value L_Small -> 3.3uH; footprint Inductor_SMD:L_0805_2012Metric_Pad1.05x1.20mm_HandSolder -> Custom_Footprints:L_0806; Part_Number C1046 -> C326343
- R32: value 4k7 -> 33k; footprint Resistor_SMD:R_0603_1608Metric -> Resistor_SMD:R_0603_1608Metric_Pad0.98x0.95mm_HandSolder; Part_Number C23162 -> (none)
- R33: value 4k7 -> 10k; footprint Resistor_SMD:R_0603_1608Metric -> Resistor_SMD:R_0603_1608Metric_Pad0.98x0.95mm_HandSolder; Part_Number C23162 -> (none)
- U3: footprint Package_SO:SO-14_3.9x8.65mm_P1.27mm -> SMD_Packages:SOIC-14_N; Part_Number (none) -> C116668
- renumbered J2 to J6
Connections:
- net +5V is gone; now on net +3.3VA: TP3.1
- net MIDI_IN is gone; now on net +3.3V: R32.1
- net MIDI_UART is gone; now on net FB: R33.1
- net +12V: now also C39.1, C40.1, U6.3 (VIN), U6.5 (EN), U6.8 (V+), U7.3 (VI)
- net +3.3VA: now also U2.4 (V+), U3.4 (V+), C41.1, J1.7 (Pin_7), J2.1 (Pin_1), J3.7 (Pin_7), J4.7 (Pin_7), L2.1, U7.8 (V+); no longer L1.2
- net -12V: now also U6.4 (V-)
- net CLOCK: now also J3.2 (Pin_2), U7.5 (+)
- net DLY_FEEDBACK: now also J2.2 (Pin_2)
- net DLY_FILTER_CV: now also J1.2 (Pin_2)
- net DLY_FILTER_POT: now also J1.3 (Pin_3)
- net DLY_MIX: now also J3.5 (Pin_5)
- net DLY_TIME_CV: now also J2.3 (Pin_3)
- net DLY_TIME_POT: now also J1.1 (Pin_1)
- net FX_FEEDBACK_CV: now also J2.4 (Pin_4)
- net FX_FEEDBACK_POT: now also J2.5 (Pin_5)
- net FX_MIX: now also J3.6 (Pin_6)
- net FX_TYPE: now also U1.78 (PC10), J3.1 (Pin_1)
- net GND: now also R33.2, C39.2, C40.2, C41.2, C42.2, J1.8 (Pin_8), J2.8 (Pin_8), J3.8 (Pin_8), J4.8 (Pin_8), J7.2 (Pin_2), J7.5 (GND), U1.6 (GND), U6.1 (GND), U7.1 (GND), U7.3 (+), U7.4 (V-)
- net IN1: now also J4.1 (Pin_1)
- net IN2: now also J4.2 (Pin_2)
- net IN3: now also J4.3 (Pin_3)
- net IN4: now also J4.4 (Pin_4)
- net LFO_BASEFREQ_CV: now also J2.6 (Pin_6)
- net LFO_BASEFREQ_POT: now also J2.7 (Pin_7)
- net LFO_RANGE: now also J1.6 (Pin_6)
- net LFO_SPEED_CV: now also J1.4 (Pin_4)
- net LFO_SPEED_POT: now also J1.5 (Pin_5)
- net OUT_AMP1: now also J4.5 (Pin_5), U6.1
- net OUT_AMP2: now also J4.6 (Pin_6), U6.7
- net PDN: now also U1.62 (PD15)
- net SWCLK: now also J7.4 (Pin_4)
- net SWIO: now also J7.3 (Pin_3)
- net USB_DM: now also U1.3 (D2_OUT)
- net USB_DP: now also U1.2 (D1_OUT)
- net at R26.1, R30.2: now also U6.6 (-)
- net at C16.1, R20.1: now also U6.5 (+)
- net at R25.1, R29.2: now also U6.2 (-)
- net at C15.1, R19.1: now also U6.3 (+)
- net at R1.1, R5.1, R6.2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: now also U7.2 (-)
- net FB: now reaches R32.2
- net FB: now also U6.4 (VFB)
- net Delay_Led_Out: now reaches U1.59 (PD12)
- net Delay_Led_Out: now also R17.1
- net FX_Led_Out: now reaches U1.60 (PD13)
- net FX_Led_Out: now also R19.1
- net Clock_Scaled: now reaches U1.80 (PC12)
- net Clock_Scaled: now also U7.6 (-), U7.7
- net +3V3 renamed +3.3V
- net +3.3V: now also L1.2, C42.1, J7.1 (Pin_1); no longer L1.1, R33.2, U2.4 (V+), U3.4 (V+)
- net DLY_FILTER renamed Delay_Filter
- net DLY_TIME renamed Delay_Time
- net FX_FEEDBACK renamed FX_Feedback
- net LFO_BASEFREQ renamed LFO_Base_Freq
- net LFO_Base_Freq: now also U7.1
- net LFO_SPEED renamed LFO_Speed
- net OUT1 renamed Audio_Out1
- net OUT2 renamed Audio_Out2
- net OUT3 renamed Audio_Out3
- net Audio_Out3: now also J8.1 (Pin_1)
- net OUT4 renamed Audio_Out4
- net Audio_Out4: now also J8.2 (Pin_2)
- new net CB: C38.2, U6.6 (VBST)
- new net D+: J7.3 (D+), U1.5 (D1_IN)
- new net D-: J7.2 (D-), U1.4 (D2_IN)
- new net DELAY_LED: J3.3 (Pin_3), R17.2
- new net FX_LED: J3.4 (Pin_4), R19.2
- new net VO: L2.2, U7.2 (VO)
- new net VSW: C38.1, L1.1, U6.2 (SW)
- no-connect marks 0 -> 53
Other:
- note added: "Analog 3.3V Supply"
- note added: "Digital 3.3V Supply"
- note removed: "UART4_RX"
- moved on the sheet: C15, C16, C19, C22, C25, C26, C27, C28, C29, C30, C31, C32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

Commit message: Started component layout
Parts:
- J1, J2, J3, J4: footprint (none) -> Connector_PinHeader_2.54mm:PinHeader_1x08_P2.54mm_Vertical
- J7: footprint (none) -> Connector_PinHeader_2.54mm:PinHeader_1x04_P2.54mm_Vertical
- J8: footprint (none) -> Connector_PinHeader_2.54mm:PinHeader_1x02_P2.54mm_Vertical
- R1, R5, R6, R7: footprint Resistors_SMD:R_0603_HandSoldering -> Resistor_SMD:R_0603_1608Metric_Pad0.98x0.95mm_HandSolder
- R17, R19: footprint Resistor_SMD:R_0603_1608Metric -> Resistor_SMD:R_0603_1608Metric_Pad0.98x0.95mm_HandSolder
- R5: renamed from R31; footprint Resistor_SMD:R_0603_1608Metric -> Resistor_SMD:R_0603_1608Metric_Pad0.98x0.95mm_HandSolder
- U3: footprint SMD_Packages:SOIC-14_N -> Package_SO:SO-14_3.9x8.65mm_P1.27mm
- U3: renamed from U6; footprint (none) -> Package_SO:SOIC-8_3.9x4.9mm_P1.27mm
- U6: renamed from U3; footprint SMD_Packages:SOIC-14_N -> Package_SO:SO-14_3.9x8.65mm_P1.27mm
- U7: footprint (none) -> Package_SO:MSOP-8_3x3mm_P0.65mm
- U7: footprint TO_SOT_Packages_SMD:SOT-223-3_TabPin2 -> Package_TO_SOT_SMD:SOT-223-3_TabPin2
- renumbered C41 to C12, C42 to C13, C19 to C18, C22 to C19, C25 to C24, C35 to C36, C36 to C37, C37 to C38, C38 to C39, C44 to C40, C39 to C41, C40 to C42, C15 to C43, C16 to C44, J6 to J5, R7 to R10, R8 to R11, R13 to R12, R14 to R13, R16 to R14, R17 to R15, R15 to R16, R18 to R17, R6 to R2, R19 to R38, R20 to R39, R25 to R40, R26 to R41, R29 to R42, R30 to R43, R9 to R6, R10 to R7, R11 to R8, R12 to R9, TP4 to TP1, TP1 to TP2, TP2 to TP3, TP3 to TP4, U1 to U2, U2 to U4, U4 to U9

Commit message: Preliminary component routing
Parts:
- removed C9: 100nF, Capacitor_SMD:C_0603_1608Metric_Pad1.08x0.95mm_HandSolder, symbol Device:C_Small
- removed RESET1: SW_Push, Custom_Footprints:SW_SPST_EVQQ2, symbol Switch:SW_Push
- added TP8: Reset, Custom_Footprints:1mm_Test_Point, symbol Connector:TestPoint
Connections:
- net Audio_Out1: now also C44.2; no longer C43.2
- net Audio_Out2: now also C43.2; no longer C44.2
- net CLOCK: now also J4.2 (Pin_2); no longer J3.2 (Pin_2)
- net DELAY_LED: now also J4.3 (Pin_3); no longer J3.3 (Pin_3)
- net Delay_Time: now also U2.31 (PA6); no longer U2.16 (PC1)
- net FX_Feedback: now also U2.24 (PA1); no longer U2.18 (PC3_C)
- net FX_LED: now also J4.4 (Pin_4); no longer J3.4 (Pin_4)
- net FX_MIX: now also U2.26 (PA3); no longer U2.17 (PC2_C)
- net FX_TYPE: now also J4.1 (Pin_1); no longer J3.1 (Pin_1)
- net IN1: now also J3.4 (Pin_4); no longer J4.1 (Pin_1)
- net IN2: now also J3.3 (Pin_3); no longer J4.2 (Pin_2)
- net IN3: now also J3.2 (Pin_2); no longer J4.3 (Pin_3)
- net IN4: now also J3.1 (Pin_1); no longer J4.4 (Pin_4)
- net LFO_RANGE: now also U2.25 (PA2); no longer U2.15 (PC0)
- net OUT_AMP1: now also J4.6 (Pin_6), R43.1, U3.7; no longer J4.5 (Pin_5), R42.1, U3.1
- net OUT_AMP2: now also J4.5 (Pin_5), R42.1, U3.1; no longer J4.6 (Pin_6), R43.1, U3.7
- net SAI2_SD_A: now also U2.15 (PC0); no longer U2.58 (PD11)
- net SAI2_SD_B: now also U2.23 (PA0); no longer U2.42 (PE11)
- net SPI1_NSS: now also U2.29 (PA4); no longer U2.77 (PA15)
- net at U2.14 (NRST): now also TP8.1
- no-connect marks 53 -> 52

Commit message: First pass signal routing of component board
Connections:
- net +3.3VA: no longer J1.7 (Pin_7)
- net CLOCK: now also J1.7 (Pin_7); no longer J4.2 (Pin_2)
- net DELAY_LED: now also J2.6 (Pin_6); no longer J4.3 (Pin_3)
- net DLY_FEEDBACK: now also J4.1 (Pin_1), U2.31 (PA6); no longer J2.2 (Pin_2), U2.35 (PB0)
- net DLY_FILTER_CV: now also J1.3 (Pin_3); no longer J1.2 (Pin_2)
- net DLY_FILTER_POT: now also J1.4 (Pin_4); no longer J1.3 (Pin_3)
- net DLY_MIX: now also J4.2 (Pin_2), U2.32 (PA7); no longer J3.5 (Pin_5), U2.34 (PC5)
- net DLY_TIME_CV: now also J1.1 (Pin_1); no longer J2.3 (Pin_3)
- net DLY_TIME_POT: now also J1.2 (Pin_2); no longer J1.1 (Pin_1)
- net Delay_Filter: now also U2.36 (PB1); no longer U2.32 (PA7)
- net Delay_Time: now also U2.35 (PB0); no longer U2.31 (PA6)
- net FX_FEEDBACK_CV: now also J2.2 (Pin_2); no longer J2.4 (Pin_4)
- net FX_FEEDBACK_POT: now also J2.3 (Pin_3); no longer J2.5 (Pin_5)
- net FX_Feedback: now also U2.34 (PC5); no longer U2.24 (PA1)
- net FX_LED: now also J2.7 (Pin_7); no longer J4.4 (Pin_4)
- net FX_MIX: now also J4.4 (Pin_4); no longer J3.6 (Pin_6)
- net FX_TYPE: now also J3.1 (Pin_1), U2.87 (PD6); no longer J4.1 (Pin_1), U2.78 (PC10)
- net IN1: now also J3.6 (Pin_6); no longer J3.4 (Pin_4)
- net IN2: now also J3.5 (Pin_5); no longer J3.3 (Pin_3)
- net IN3: now also J3.4 (Pin_4); no longer J3.2 (Pin_2)
- net IN4: now also J3.3 (Pin_3); no longer J3.1 (Pin_1)
- net LFO_BASEFREQ_CV: now also J1.5 (Pin_5); no longer J2.6 (Pin_6)
- net LFO_BASEFREQ_POT: now also J1.6 (Pin_6); no longer J2.7 (Pin_7)
- net LFO_Base_Freq: now also U2.24 (PA1); no longer U2.36 (PB1)
- net LFO_RANGE: now also J3.2 (Pin_2); no longer J1.6 (Pin_6)
- net LFO_SPEED_CV: now also J2.5 (Pin_5); no longer J1.4 (Pin_4)
- net LFO_SPEED_POT: now also J2.4 (Pin_4); no longer J1.5 (Pin_5)
Changed lines of the file:
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@@
   (no_connect (at 82.55 121.92))
   (no_connect (at 82.55 160.02))
+  (no_connect (at 82.55 157.48))
   (no_connect (at 82.55 127))
   (no_connect (at 39.37 167.64))
   (no_connect (at 82.55 99.06))
-  (no_connect (at 39.37 147.32))
   (no_connect (at 82.55 86.36))
   (no_connect (at 39.37 114.3))
@@
     (stroke (width 0) (type default))
   )
+  (wire (pts (xy 34.29 147.32) (xy 39.37 147.32))
+    (stroke (width 0) (type default))
+  )
   (wire (pts (xy 302.26 99.06) (xy 302.26 105.41))
     (stroke (width 0) (type default))
@@
     (stroke (width 0) (type solid))
   )
-  (wire (pts (xy 85.09 157.48) (xy 82.55 157.48))
-    (stroke (width 0) (type default))
-  )
   (wire (pts (xy 132.08 252.73) (xy 132.08 255.27))
     (stroke (width 0) (type default))
@@
     (effects (font (size 1.27 1.27)) (justify left bottom))
   )
-  (label "LFO_Base_Freq" (at 85.09 93.98 0) (fields_autoplaced)
+  (label "LFO_Base_Freq" (at 85.09 50.8 0) (fields_autoplaced)
     (effects (font (size 1.27 1.27)) (justify left bottom))
   )
@@
     (effects (font (size 1.27 1.27)) (justify left bottom))
   )
-  (label "DLY_FILTER_CV" (at 214.63 219.71 0) (fields_autoplaced)
+  (label "DLY_FILTER_CV" (at 214.63 222.25 0) (fields_autoplaced)
     (effects (font (size 1.27 1.27)) (justify left bottom))
   )
@@
     (effects (font (size 1.27 1.27)) (justify left bottom))
   )
-  (label "DLY_FEEDBACK" (at 85.09 91.44 0) (fields_autoplaced)
+  (label "DLY_FEEDBACK" (at 85.09 63.5 0) (fields_autoplaced)
     (effects (font (size 1.27 1.27)) (justify left bottom))
   )
@@
     (effects (font (size 1.27 1.27)) (justify left bottom))
   )
-  (label "DLY_TIME_CV" (at 248.92 222.25 0) (fields_autoplaced)
-    (effects (font (size 1.27 1.27)) (justify left bottom))
-  )
-  (label "FX_TYPE" (at 85.09 157.48 0) (fields_autoplaced)
-    (effects (font (size 1.27 1.27)) (justify left bottom))
+  (label "DLY_TIME_CV" (at 214.63 217.17 0) (fields_autoplaced)
+    (effects (font (size 1.27 1.27)) (justify left bottom))
+  )
+  (label "FX_TYPE" (at 34.29 147.32 180) (fields_autoplaced)
+    (effects (font (size 1.27 1.27)) (justify right bottom))
   )
   (label "SWIO" (at 309.88 234.95 0) (fields_autoplaced)
@@
     (effects (font (size 1.27 1.27)) (justify right bottom))
   )
-  (label "DLY_MIX" (at 214.63 264.16 0) (fields_autoplaced)
-    (effects (font (size 1.27 1.27)) (justify left bottom))
-  )
-  (label "FX_LED" (at 248.92 260.35 0) (fields_autoplaced)
-    (effects (font (size 1.27 1.27)) (justify left bottom))
-  )
-  (label "LFO_BASEFREQ_CV" (at 248.92 229.87 0) (fields_autoplaced)
+  (label "DLY_MIX" (at 248.92 255.27 0) (fields_autoplaced)
+    (effects (font (size 1.27 1.27)) (justify left bottom))
+  )
+  (label "FX_LED" (at 248.92 232.41 0) (fields_autoplaced)
+    (effects (font (size 1.27 1.27)) (justify left bottom))
+  )
+  (label "LFO_BASEFREQ_CV" (at 214.63 227.33 0) (fields_autoplaced)
     (effects (font (size 1.27 1.27)) (justify left bottom))
   )
@@
     (effects (font (size 1.27 1.27)) (justify left bottom))
   )
-  (label "DELAY_LED" (at 248.92 257.81 0) (fields_autoplaced)
+  (label "DELAY_LED" (at 248.92 229.87 0) (fields_autoplaced)
     (effects (font (size 1.27 1.27)) (justify left bottom))
   )
@@
     (effects (font (size 1.27 1.27)) (justify right bottom))
   )
-  (label "IN1" (at 214.63 261.62 0) (fields_autoplaced)
-    (effects (font (size 1.27 1.27)) (justify left bottom))
-  )
-  (label "LFO_BASEFREQ_POT" (at 248.92 232.41 0) (fields_autoplaced)
+  (label "IN1" (at 214.63 266.7 0) (fields_autoplaced)
+    (effects (font (size 1.27 1.27)) (justify left bottom))
+  )
+  (label "LFO_BASEFREQ_POT" (at 214.63 229.87 0) (fields_autoplaced)
     (effects (font (size 1.27 1.27)) (justify left bottom))
   )
@@
     (effects (font (size 1.27 1.27)) (justify left bottom))
   )
-  (label "DLY_FEEDBACK" (at 248.92 219.71 0) (fields_autoplaced)
+  (label "DLY_FEEDBACK" (at 248.92 252.73 0) (fields_autoplaced)
     (effects (font (size 1.27 1.27)) (justify left bottom))
   )
@@
     (effects (font (size 1.27 1.27)) (justify left bottom))
   )
-  (label "IN3" (at 214.63 256.54 0) (fields_autoplaced)
+  (label "IN3" (at 214.63 261.62 0) (fields_autoplaced)
     (effects (font (size 1.27 1.27)) (justify left bottom))
   )
@@
     (effects (font (size 1.27 1.27)) (justify right bottom))
   )
-  (label "DLY_FILTER_POT" (at 214.63 222.25 0) (fields_autoplaced)
+  (label "DLY_FILTER_POT" (at 214.63 224.79 0) (fields_autoplaced)
     (effects (font (size 1.27 1.27)) (justify left bottom))
   )
@@
     (effects (font (size 1.27 1.27)) (justify left bottom))
   )
-  (label "FX_FEEDBACK_POT" (at 248.92 227.33 0) (fields_autoplaced)
-    (effects (font (size 1.27 1.27)) (justify left bottom))
-  )
-  (label "FX_FEEDBACK_CV" (at 248.92 224.79 0) (fields_autoplaced)
+  (label "FX_FEEDBACK_POT" (at 248.92 222.25 0) (fields_autoplaced)
+    (effects (font (size 1.27 1.27)) (justify left bottom))
+  )
+  (label "FX_FEEDBACK_CV" (at 248.92 219.71 0) (fields_autoplaced)
     (effects (font (size 1.27 1.27)) (justify left bottom))
   )
@@
     (effects (font (size 1.27 1.27)) (justify left bottom))
   )
-  (label "DLY_MIX" (at 85.09 144.78 0) (fields_autoplaced)
+  (label "DLY_MIX" (at 85.09 66.04 0) (fields_autoplaced)
     (effects (font (size 1.27 1.27)) (justify left bottom))
   )
@@
     (effects (font (size 1.27 1.27)) (justify right bottom))
   )
-  (label "CLOCK" (at 248.92 255.27 0) (fields_autoplaced)
+  (label "CLOCK" (at 214.63 232.41 0) (fields_autoplaced)
     (effects (font (size 1.27 1.27)) (justify left bottom))
   )
@@
     (effects (font (size 1.27 1.27)) (justify left bottom))
   )
-  (label "DLY_TIME_POT" (at 214.63 217.17 0) (fields_autoplaced)
-    (effects (font (size 1.27 1.27)) (justify left bottom))
-  )
-  (label "IN2" (at 214.63 259.08 0) (fields_autoplaced)
+  (label "DLY_TIME_POT" (at 214.63 219.71 0) (fields_autoplaced)
+    (effects (font (size 1.27 1.27)) (justify left bottom))
+  )
+  (label "IN2" (at 214.63 264.16 0) (fields_autoplaced)
     (effects (font (size 1.27 1.27)) (justify left bottom))
   )
@@
     (effects (font (size 1.27 1.27)) (justify left bottom))
   )
-  (label "FX_Feedback" (at 85.09 50.8 0) (fields_autoplaced)
+  (label "FX_Feedback" (at 85.09 144.78 0) (fields_autoplaced)
     (effects (font (size 1.27 1.27)) (justify left bottom))
   )
@@
     (effects (font (size 1.27 1.27)) (justify right bottom))
   )
-  (label "Delay_Filter" (at 85.09 66.04 0) (fields_autoplaced)
+  (label "Delay_Filter" (at 85.09 93.98 0) (fields_autoplaced)
     (effects (font (size 1.27 1.27)) (justify left bottom))
   )
@@
     (effects (font (size 1.27 1.27)) (justify right bottom))
   )
-  (label "LFO_SPEED_CV" (at 214.63 224.79 0) (fields_autoplaced)
+  (label "LFO_SPEED_CV" (at 248.92 227.33 0) (fields_autoplaced)
     (effects (font (size 1.27 1.27)) (justify left bottom))
   )
@@
     (effects (font (size 1.27 1.27)) (justify left bottom))
   )
-  (label "FX_TYPE" (at 248.92 252.73 0) (fields_autoplaced)
+  (label "FX_TYPE" (at 214.63 254 0) (fields_autoplaced)
     (effects (font (size 1.27 1.27)) (justify left bottom))
   )
@@
     (effects (font (size 1.27 1.27)) (justify left bottom))
   )
-  (label "Delay_Time" (at 85.09 63.5 0) (fields_autoplaced)
+  (label "Delay_Time" (at 85.09 91.44 0) (fields_autoplaced)
     (effects (font (size 1.27 1.27)) (justify left bottom))
   )
@@
     (effects (font (size 1.27 1.27)) (justify left bottom))
   )
-  (label "LFO_SPEED_POT" (at 214.63 227.33 0) (fields_autoplaced)
+  (label "LFO_SPEED_POT" (at 248.92 224.79 0) (fields_autoplaced)
     (effects (font (size 1.27 1.27)) (justify left bottom))
   )
@@
     (effects (font (size 1.27 1.27)) (justify right bottom))
   )
-  (label "FX_MIX" (at 214.63 266.7 0) (fields_autoplaced)
-    (effects (font (size 1.27 1.27)) (justify left bottom))
-  )
-  (label "IN4" (at 214.63 254 0) (fields_autoplaced)
+  (label "FX_MIX" (at 248.92 260.35 0) (fields_autoplaced)
+    (effects (font (size 1.27 1.27)) (justify left bottom))
+  )
+  (label "IN4" (at 214.63 259.08 0) (fields_autoplaced)
     (effects (font (size 1.27 1.27)) (justify left bottom))
   )
@@
     (effects (font (size 1.27 1.27)) (justify right bottom))
   )
-  (label "LFO_RANGE" (at 214.63 229.87 0) (fields_autoplaced)
+  (label "LFO_RANGE" (at 214.63 256.54 0) (fields_autoplaced)
     (effects (font (size 1.27 1.27)) (justify left bottom))
   )
@@
         )
       )
-    )
-  )
-  (symbol (lib_id "power:+3.3VA") (at 214.63 232.41 270) (unit 1)
-    (in_bom yes) (on_board yes) (dnp no)
-    (property "Reference" "#PWR04" (at 210.82 232.41 0)
-      (effects (font (size 1.27 1.27)) hide)
-    )
-    (property "Value" "+3.3VA" (at 218.44 231.14 90)
-      (effects (font (size 1.27 1.27)) (justify left))
-    )
-    (property "Footprint" "" (at 214.63 232.41 0)
-      (effects (font (size 1.27 1.27)) hide)
-    )
-    (property "Datasheet" "" (at 214.63 232.41 0)
-      (effects (font (size 1.27 1.27)) hide)
-    )
-    (pin "1")
-    (instances
-      (project "Punck_Components"
-        (path "/863a2fa5-cc81-43c1-8f46-cd3e70a7a26b"
-          (reference "#PWR04") (unit 1)
-        )
-      )
-      (project "QuadMod Components"
-        (path "/d7d98a4b-a059-4480-8e77-1d52297d5f57"
-          (reference "#PWR073") (unit 1)
-        )
-      )
