File: Hardware/QuadMod_Panel.kicad_pcb (KiCad board)
At the start: 2 copper layers, 60.8 x 128.5 mm, 24 parts

Commit message: Work on panel
Parts:
- added MIX: Alpha_9mm_pot_hole, Custom_Footprints:Alpha_9mm_pot_hole, F.Cu at (111.0, 112.0)
- added REF**: RJ45_Amphenol_RJHSE-3080_Mounting_Hole, Custom_Footprints:RJ45_Amphenol_RJHSE-3080_Mounting_Hole, F.Cu at (63.0, 147.0)
- added kibuzzard-65B27F4A: G***, kibuzzard-65B27F4A, F.Cu at (122.5, 54.5)
- added kibuzzard-65B28018: G***, kibuzzard-65B28018, F.Cu at (147.0, 88.0)
- moved Ref** 126.2 mm to (280.0, 134.0)
- moved Ref** 126.2 mm to (270.0, 134.0)
- moved MIX 37.1 mm to (133.0, 66.9)
- moved MIX 36.2 mm to (133.0, 87.5)
- moved TYPE 33.9 mm to (133.0, 112.0)
- moved Ref** 27.8 mm to (163.0, 152.0)
- moved Ref** 26.3 mm to (149.0, 134.0)
- moved Ref** 23.8 mm to (149.0, 152.0)
- moved Ref** 18.8 mm to (107.0, 134.0)
- moved Ref** 15.0 mm to (121.0, 134.0)
- moved REF** 11.5 mm to (119.0, 153.0)
- moved Ref** 11.3 mm to (135.0, 134.0)
- moved MIX 10.9 mm to (111.0, 87.6)
- moved Ref** 10.0 mm to (163.2, 43.9)
- moved Ref** 10.0 mm to (163.2, 166.4)
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Other:
- board size 60.8 x 128.5 mm -> 70.8 x 128.5 mm
- board text added: "Audio In"
- board text added: "Base Freq"
- board text added: "Flanger"
- board text added: "Freq"
- board text added: "Left"
- board text added: "Mix"
- board text added: "Phaser"
- board text added: "Range"
- board text added: "Right"
- board text added: "Speed"
- board text removed: "Delay Mix"
- board text removed: "Delay Time"
- board text removed: "LFO Base Frequency"
- board text removed: "LFO Range"
- board text removed: "LFO Speed"
- board text removed: "Modulation"

Commit message: Updates to Panel
Parts:
- removed the REF** at (63.0, 147.0)
- removed the Ref** at (280.0, 134.0)
- removed the Ref** at (270.0, 134.0)
- removed kibuzzard-65B27F4A: G***, kibuzzard-65B27F4A
- removed kibuzzard-65B28018: G***, kibuzzard-65B28018
- added kibuzzard-65B29BBA: G***, kibuzzard-65B29BBA, F.Cu at (157.0, 140.0)
- added kibuzzard-65B29BCB: G***, kibuzzard-65B29BCB, F.Cu at (157.0, 119.0)
- added kibuzzard-65B29CC1: G***, kibuzzard-65B29CC1, F.Cu at (157.0, 98.0)
- added kibuzzard-65B29D47: G***, kibuzzard-65B29D47, F.Cu at (156.5, 54.0)
- added kibuzzard-65B29D82: G***, kibuzzard-65B29D82, F.Cu at (122.0, 54.0)
- added kibuzzard-65B29E0F: G***, kibuzzard-65B29E0F, F.Cu at (111.0, 77.0)
- added kibuzzard-65B29E0F: G***, kibuzzard-65B29E0F, F.Cu at (157.0, 77.0)
- added kibuzzard-65B29E34: G***, kibuzzard-65B29E34, F.Cu at (111.0, 119.0)
- added kibuzzard-65B29E5A: G***, kibuzzard-65B29E5A, F.Cu at (111.0, 98.0)
- added kibuzzard-65B29EC8: G***, kibuzzard-65B29EC8, F.Cu at (133.0, 119.0)
- added kibuzzard-65B29EDF: G***, kibuzzard-65B29EDF, F.Cu at (133.0, 98.0)
- added kibuzzard-65B2A755: G***, kibuzzard-65B2A755, F.Cu at (133.0, 62.0)
- added kibuzzard-65B2A761: G***, kibuzzard-65B2A761, F.Cu at (133.0, 74.5)
- moved MIX 44.0 mm to (111.0, 68.0)
- moved TYPE 44.0 mm to (133.0, 68.0)
- moved Ref** 25.5 mm to (137.5, 151.0)
- moved Ref** 23.0 mm to (126.0, 151.0)
- moved MIX 22.5 mm to (133.0, 110.0)
- moved MIX 22.4 mm to (111.0, 110.0)
- moved MIX 22.1 mm to (133.0, 89.0)
- moved MIX 22.0 mm to (111.0, 89.0)
- moved Ref** 17.1 mm to (150.5, 151.0)
- moved Ref** 17.0 mm to (163.0, 151.0)
- moved MIX 12.0 mm to (157.0, 131.0)
- moved MIX 12.0 mm to (157.0, 110.0)
- moved MIX 11.0 mm to (157.0, 89.0)
- moved MIX 9.75 mm to (157.0, 68.0)
- moved REF** 9.34 mm to (110.0, 150.5)
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Other:
- board text added: "OUT L/R"
- board text added: "Regen"
- board text removed: "Base Freq"
- board text removed: "Delay"
- board text removed: "Feedback"
- board text removed: "Flanger"
- board text removed: "Left"
- board text removed: "Mix"
- board text removed: "Phaser"
- board text removed: "Range"
- board text removed: "Right"

Commit message: First draft of panel completed
Parts:
- removed kibuzzard-65B29EDF: G***, kibuzzard-65B29EDF
- added kibuzzard-65B38E0B: G***, kibuzzard-65B38E0B, F.Cu at (133.0, 98.0)
- added kibuzzard-65B38FE8: G***, kibuzzard-65B38FE8, F.Cu at (135.3, 167.3)
- moved kibuzzard-65B29E0F 63.5 mm to (157.0, 140.5)
- moved kibuzzard-65B29BBA 63.0 mm to (157.0, 77.0)
- moved G*** 0.94 mm to (135.5, 45.2)

Commit message: Cleaned up schematic
Other:
- board text added: "L OUT R"
- board text removed: "Mountjoy Modular"
- board text removed: "OUT L/R"
Changed lines of the file:
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@@
     (effects (font (size 2 2) (thickness 0.3)))
   )
-  (gr_text "OUT L/R" (at 132 159) (layer "F.Mask")
+  (gr_text "L  OUT  R" (at 132 159) (layer "F.Mask")
     (effects (font (size 2 2) (thickness 0.3)))
   )
@@
     (effects (font (size 2 2) (thickness 0.3)))
   )
-  (gr_text "Mountjoy Modular" (at 136 178) (layer "F.Mask")
-    (effects (font (size 2 2) (thickness 0.3)))
-  )

Commit message: First draft of control board
Parts:
- moved Ref** 0.90 mm to (108.4, 131.0)
Changed lines of the file:
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@@
   )
   (footprint "Custom_Footprints:Thonkiconn_Socket_MountingHole_6mm" (layer "F.Cu")
-    (at 107.5 131 180)
+    (at 108.4 131 180)
     (descr "Mounting Hole 6mm, no annular")
     (tags "mounting hole 6mm no annular")

Commit message: Clean up of schematics and PCBS
Parts:
- removed kibuzzard-65B38FE8: G***, kibuzzard-65B38FE8
- added kibuzzard-65BBC0F3: G***, kibuzzard-65BBC0F3, F.Cu at (135.3, 167.4)
- TYPE: footprint Custom_Footprints:Sub_Miniature_Switch_MountingHole_5mm -> Custom_Footprints:Miniature_Switch_MountingHole_6.35mm
- moved kibuzzard-65B2A755 0.50 mm to (133.0, 61.5)
- moved kibuzzard-65B2A761 0.20 mm to (133.0, 74.7)
Other:
- board text added: "Time"
- board text removed: "Clock"
